Commit message: changed gripper transmission

File: ur_rh_description/urdf/common.gazebo.xacro (robot description, xacro)
@@ -5,4 +5,13 @@
       <robotNamespace>/</robotNamespace>
       <robotSimType>gazebo_ros_control/DefaultRobotHWSim</robotSimType>
+    </plugin>
+    <!-- loading plugin: mimic joints works in gazebo now -->
+    <plugin name="gazebo_gripper_ros_control" filename="libroboticsgroup_gazebo_mimic_joint_plugin.so">
+      <joint>rh_p12_rn_a</joint>
+      <mimicJoint>rh_r2</mimicJoint>
+      <mimicJoint>rh_l1</mimicJoint>
+      <mimicJoint>rh_l2</mimicJoint>
+      <multiplier>1.0</multiplier>
+      <offset>0.0</offset>
     </plugin>
 <!--

File: ur_rh_description/urdf/rh_p12_rn_a.transmission.xacro (robot description, xacro)
@@ -4,38 +4,8 @@
     <type>transmission_interface/SimpleTransmission</type>
     <joint name="rh_p12_rn_a">
-      <hardwareInterface>hardware_interface/EffortJointInterface</hardwareInterface>
+      <hardwareInterface>hardware_interface/PositionJointInterface</hardwareInterface>
     </joint>
     <actuator name="motor_r1">
-      <hardwareInterface>hardware_interface/EffortJointInterface</hardwareInterface>
-      <mechanicalReduction>1</mechanicalReduction>
-    </actuator>
-  </transmission>
-  <transmission name="tran_r2">
-    <type>transmission_interface/SimpleTransmission</type>
-    <joint name="rh_r2">
-      <hardwareInterface>hardware_interface/EffortJointInterface</hardwareInterface>
-    </joint>
-    <actuator name="motor_r2">
-      <hardwareInterface>hardware_interface/EffortJointInterface</hardwareInterface>
-      <mechanicalReduction>1</mechanicalReduction>
-    </actuator>
-  </transmission>
-  <transmission name="tran_l1">
-    <type>transmission_interface/SimpleTransmission</type>
-    <joint name="rh_l1">
-      <hardwareInterface>hardware_interface/EffortJointInterface</hardwareInterface>
-    </joint>
-    <actuator name="motor_l1">
-      <hardwareInterface>hardware_interface/EffortJointInterface</hardwareInterface>
-      <mechanicalReduction>1</mechanicalReduction>
-    </actuator>
-  </transmission>
-  <transmission name="tran_l2">
-    <type>transmission_interface/SimpleTransmission</type>
-    <joint name="rh_l2">
-      <hardwareInterface>hardware_interface/EffortJointInterface</hardwareInterface>
-    </joint>
-    <actuator name="motor_l2">
-      <hardwareInterface>hardware_interface/EffortJointInterface</hardwareInterface>
+      <hardwareInterface>hardware_interface/PositionJointInterface</hardwareInterface>
       <mechanicalReduction>1</mechanicalReduction>
     </actuator>

Commit message: fixed gripper bug

File: ur_rh_description/urdf/common.gazebo.xacro (robot description, xacro)
@@ -10,5 +10,15 @@
       <joint>rh_p12_rn_a</joint>
       <mimicJoint>rh_r2</mimicJoint>
+      <multiplier>1.0</multiplier>
+      <offset>0.0</offset>
+    </plugin>
+    <plugin name="gazebo_gripper_ros_control" filename="libroboticsgroup_gazebo_mimic_joint_plugin.so">
+      <joint>rh_p12_rn_a</joint>
       <mimicJoint>rh_l1</mimicJoint>
+      <multiplier>1.0</multiplier>
+      <offset>0.0</offset>
+    </plugin>
+    <plugin name="gazebo_gripper_ros_control" filename="libroboticsgroup_gazebo_mimic_joint_plugin.so">
+      <joint>rh_p12_rn_a</joint>
       <mimicJoint>rh_l2</mimicJoint>
       <multiplier>1.0</multiplier>

File: ur_rh_description/urdf/rh_p12_rn_a.urdf.xacro (robot description, xacro)
@@ -63,4 +63,5 @@
     <axis xyz="-1 0 0"/>
     <limit velocity="6.5" effort="1000" lower="0.0" upper="1.0" />
+    <mimic joint="rh_p12_rn_a" multiplier="1"/>
     <dynamics damping="0.7"/>
   </joint>
@@ -94,4 +95,5 @@
     <axis xyz="-1 0 0"/>
     <limit velocity="6.5" effort="1000" lower="0.0" upper="1.1" />
+    <mimic joint="rh_p12_rn_a" multiplier="1"/>
     <dynamics damping="0.7"/>
   </joint>
@@ -125,4 +127,5 @@
     <axis xyz="1 0 0"/>
     <limit velocity="6.5" effort="1000" lower="0.0" upper="1.0" />
+    <mimic joint="rh_p12_rn_a" multiplier="1"/>
     <dynamics damping="0.7"/>
   </joint>

File: ur_rh_description/urdf/ur_rh_robot.urdf.xacro (robot description, xacro)
@@ -3,5 +3,5 @@
        name="ur_rh" >
   <!-- common stuff -->
-  <xacro:include filename="$(find ur_e_description)/urdf/common.gazebo.xacro" />
+  <xacro:include filename="$(find ur_rh_description)/urdf/common.gazebo.xacro" />
   <!-- ur5e -->
   <xacro:include filename="$(find ur_e_description)/urdf/ur5e.urdf.xacro" />
